Commit message: URDF improvements

File: urdf/drivebase.xacro (robot description, xacro)
@@ -1,23 +1,20 @@
 <?xml version="1.0"?>
-<robot xmlns:xacro="http://www.ros.org/wiki/xacro" >
+<robot xmlns:xacro="http://www.ros.org/wiki/xacro">
     <!-- Imports -->
+    <xacro:include filename="params.xacro" />
     <xacro:include filename="wheels.xacro" />
-    <!-- Parameters -->
-    <xacro:property name="chassis_width" value="0.43" />
-    <xacro:property name="chassis_length" value="0.55" />
-    <xacro:property name="chassis_height" value="0.25" />
-    <xacro:property name="chassis_X_offset" value="-0.1" />
-    <xacro:property name="chassis_Z_offset" value="0.08" />
-    <xacro:property name="drive_wheels_Y_spacing" value="0.46" />
-    <xacro:property name="caster_wheels_F_Y_spacing" value="0.52" />
-    <xacro:property name="caster_wheels_R_Y_spacing" value="0.405" />
-    <xacro:property name="caster_wheels_F_X_offset" value="0.35" />
-    <xacro:property name="caster_wheels_R_X_offset" value="-0.4" />
-    <!-- Material declaration -->
+    <xacro:include filename="inertial_macros.xacro" />
+    <!-- Materials -->
     <material name="plastic_shell">
         <color rgba="0 0 1 1" />
     </material>
     <!-- Base link -->
+    <link name="base_footprint"></link>
     <link name="base_link"></link>
+    <joint name="footprint_joint" type="fixed">
+        <parent link="base_footprint"/>
+        <child link="base_link"/>
+        <origin xyz="0 0 ${drive_wheel_radius}"/>
+    </joint>
     <!-- Chassis -->
     <link name="chassis">
@@ -29,4 +26,13 @@
         <material name="plastic_shell"/>
     </visual>
+        <collision>
+            <origin xyz="0 0 0"/>
+            <geometry>
+                <box size="${chassis_length} ${chassis_width} ${chassis_height}"/>
+            </geometry>
+        </collision>
+        <xacro:inertial_box mass="50.0" x="${chassis_length}" y="${chassis_width}" z="${chassis_height}">
+            <origin xyz="0 0 0" rpy="0 0 0" />
+        </xacro:inertial_box>
     </link>
     <joint name="chassis_joint" type="fixed">
@@ -37,5 +43,5 @@
     <!-- Drive Wheels -->
     <xacro:drive_wheel name="drive_wheel_L"></xacro:drive_wheel>
-    <joint name="drive_wheel_joint_L" type="continuous">
+    <joint name="drive_wheel_L_joint" type="continuous">
         <parent link="base_link"/>
         <child link="drive_wheel_L"/>
@@ -44,5 +50,5 @@
     </joint>
     <xacro:drive_wheel name="drive_wheel_R"></xacro:drive_wheel>
-    <joint name="drive_wheel_joint_R" type="continuous">
+    <joint name="drive_wheel_R_joint" type="continuous">
         <parent link="base_link"/>
         <child link="drive_wheel_R"/>
@@ -52,10 +58,10 @@
     <!-- Caster Wheels -->
     <xacro:caster_wheel name="caster_wheel_FL"></xacro:caster_wheel>
-    <joint name="caster_wheel_joint_FL" type="fixed">
+    <joint name="caster_wheel_FL_joint" type="fixed">
         <parent link="base_link"/>
         <child link="caster_wheel_FL"/>
         <origin xyz="${caster_wheels_F_X_offset} ${caster_wheels_F_Y_spacing/2} ${-drive_wheel_radius + caster_wheel_radius + caster_wheel_Z_offset}" rpy="0 0 0" />
     </joint>
-    <xacro:caster_wheel name="caster_wheel_FR"></xacro:caster_wheel>
+    <xacro:caster_wheel name="caster_wheel_FR_joint"></xacro:caster_wheel>
     <joint name="caster_wheel_joint_FR" type="fixed">
         <parent link="base_link"/>
@@ -64,5 +70,5 @@
     </joint>
     <xacro:caster_wheel name="caster_wheel_RL"></xacro:caster_wheel>
-    <joint name="caster_wheel_joint_RL" type="fixed">
+    <joint name="caster_wheel_RL_joint" type="fixed">
         <parent link="base_link"/>
         <child link="caster_wheel_RL"/>
@@ -70,5 +76,5 @@
     </joint>
     <xacro:caster_wheel name="caster_wheel_RR"></xacro:caster_wheel>
-    <joint name="caster_wheel_joint_RR" type="fixed">
+    <joint name="caster_wheel_RR_joint" type="fixed">
         <parent link="base_link"/>
         <child link="caster_wheel_RR"/>

File: urdf/wheels.xacro (robot description, xacro)
@@ -1,12 +1,7 @@
 <?xml version="1.0"?>
 <robot xmlns:xacro="http://www.ros.org/wiki/xacro">
-    <!-- Parameters -->
-    <xacro:property name="drive_wheel_radius" value="0.17" /> <!-- TODO: Calibrate Drive wheel radius -->
-    <xacro:property name="drive_wheel_thickness" value="0.075" />
-    <xacro:property name="caster_wheel_radius" value="0.075" /> <!-- TODO: Calibrate Drive wheel radius -->
-    <xacro:property name="caster_wheel_thickness" value="0.05" />
-    <xacro:property name="caster_wheel_X_offset" value="0.05" />
-    <xacro:property name="caster_wheel_Z_offset" value="0.09" />
-    <!-- Material declaration -->
+    <!-- Imports -->
+    <xacro:include filename="params.xacro" />
+    <!-- Materials -->
     <material name="wheel_rubber">
         <color rgba="0.8 0.8 0.8 1" />
@@ -23,4 +18,13 @@
                 <material name="wheel_rubber" />
             </visual>
+            <collision>
+                <origin xyz="0 ${drive_wheel_thickness/2} 0" rpy="-${pi/2} 0 0" />
+                <geometry>
+                    <cylinder radius="${drive_wheel_radius}" length="${drive_wheel_thickness}" />
+                </geometry>
+            </collision>
+            <xacro:inertial_cylinder mass="2.0" radius="${drive_wheel_radius}" length="${drive_wheel_thickness}">
+                <origin xyz="0 ${drive_wheel_thickness/2} 0" rpy="-${pi/2} 0 0" />
+            </xacro:inertial_cylinder>
         </link>
     </xacro:macro>
@@ -35,4 +39,13 @@
                 <material name="wheel_rubber" />
             </visual>
+            <collision>
+                <origin xyz="-${caster_wheel_X_offset} 0 -${caster_wheel_Z_offset}" rpy="-${pi/2} 0 0" />
+                <geometry>
+                    <cylinder radius="${caster_wheel_radius}" length="${caster_wheel_thickness}"/>
+                </geometry>
+            </collision>
+            <xacro:inertial_cylinder mass="1.0" radius="${caster_wheel_radius}" length="${caster_wheel_thickness}">
+                <origin xyz="-${caster_wheel_X_offset} 0 -${caster_wheel_Z_offset}" rpy="-${pi/2} 0 0" />
+            </xacro:inertial_cylinder>
         </link>
     </xacro:macro>

Commit message: Add and configure gazebo

File: urdf/drivebase.xacro (robot description, xacro)
@@ -19,11 +19,11 @@
     <!-- Chassis -->
     <link name="chassis">
-    <visual>
-        <origin xyz="0 0 0"/>
-        <geometry>
-            <box size="${chassis_length} ${chassis_width} ${chassis_height}"/>
-        </geometry>
-        <material name="plastic_shell"/>
-    </visual>
+        <visual>
+            <origin xyz="0 0 0"/>
+            <geometry>
+                <box size="${chassis_length} ${chassis_width} ${chassis_height}"/>
+            </geometry>
+            <material name="plastic_shell"/>
+        </visual>
         <collision>
             <origin xyz="0 0 0"/>
@@ -61,5 +61,5 @@
         <parent link="base_link"/>
         <child link="caster_wheel_FL"/>
-        <origin xyz="${caster_wheels_F_X_offset} ${caster_wheels_F_Y_spacing/2} ${-drive_wheel_radius + caster_wheel_radius + caster_wheel_Z_offset}" rpy="0 0 0" />
+        <origin xyz="${caster_wheels_F_X_offset} ${caster_wheels_F_Y_spacing/2} ${-drive_wheel_radius + caster_wheel_radius + caster_wheel_Z_offset + 0.01}" rpy="0 0 0" />
     </joint>
     <xacro:caster_wheel name="caster_wheel_FR_joint"></xacro:caster_wheel>
@@ -67,5 +67,5 @@
         <parent link="base_link"/>
         <child link="caster_wheel_FR"/>
-        <origin xyz="${caster_wheels_F_X_offset} -${caster_wheels_F_Y_spacing/2} ${-drive_wheel_radius + caster_wheel_radius + caster_wheel_Z_offset}" rpy="0 0 0" />
+        <origin xyz="${caster_wheels_F_X_offset} -${caster_wheels_F_Y_spacing/2} ${-drive_wheel_radius + caster_wheel_radius + caster_wheel_Z_offset + 0.01}" rpy="0 0 0" />
     </joint>
     <xacro:caster_wheel name="caster_wheel_RL"></xacro:caster_wheel>
@@ -73,5 +73,5 @@
         <parent link="base_link"/>
         <child link="caster_wheel_RL"/>
-        <origin xyz="${caster_wheels_R_X_offset} ${caster_wheels_R_Y_spacing/2} ${-drive_wheel_radius + caster_wheel_radius + caster_wheel_Z_offset}" rpy="0 0 0" />
+        <origin xyz="${caster_wheels_R_X_offset} ${caster_wheels_R_Y_spacing/2} ${-drive_wheel_radius + caster_wheel_radius + caster_wheel_Z_offset + 0.01}" rpy="0 0 0" />
     </joint>
     <xacro:caster_wheel name="caster_wheel_RR"></xacro:caster_wheel>
@@ -79,5 +79,5 @@
         <parent link="base_link"/>
         <child link="caster_wheel_RR"/>
-        <origin xyz="${caster_wheels_R_X_offset} -${caster_wheels_R_Y_spacing/2} ${-drive_wheel_radius + caster_wheel_radius + caster_wheel_Z_offset}" rpy="0 0 0" />
+        <origin xyz="${caster_wheels_R_X_offset} -${caster_wheels_R_Y_spacing/2} ${-drive_wheel_radius + caster_wheel_radius + caster_wheel_Z_offset + 0.01}" rpy="0 0 0" />
     </joint>
 </robot>

File: urdf/robot.urdf.xacro (robot description, xacro)
@@ -2,3 +2,4 @@
 <robot xmlns:xacro="http://www.ros.org/wiki/xacro"  name="robot">
     <xacro:include filename="drivebase.xacro" />
+    <xacro:include filename="gazebo_control.xacro" />
 </robot>

Commit message: Improve ros2_controls with Gazebo

File: urdf/drivebase.xacro (robot description, xacro)
@@ -63,6 +63,6 @@
         <origin xyz="${caster_wheels_F_X_offset} ${caster_wheels_F_Y_spacing/2} ${-drive_wheel_radius + caster_wheel_radius + caster_wheel_Z_offset + 0.01}" rpy="0 0 0" />
     </joint>
-    <xacro:caster_wheel name="caster_wheel_FR_joint"></xacro:caster_wheel>
-    <joint name="caster_wheel_joint_FR" type="fixed">
+    <xacro:caster_wheel name="caster_wheel_FR"></xacro:caster_wheel>
+    <joint name="caster_wheel_FR_joint" type="fixed">
         <parent link="base_link"/>
         <child link="caster_wheel_FR"/>

File: urdf/gz_ros2_control.xacro (robot description, xacro)
@@ -25,5 +25,5 @@
     <gazebo>
         <plugin filename="gz_ros2_control-system" name="gz_ros2_control::GazeboSimROS2ControlPlugin">
-            <parameters>$(find luggage_av)/gazebo/dd_velocity_controller.yaml</parameters>
+            <parameters>$(find luggage_av)/parameters/gz_ros2_control.yaml</parameters>
         </plugin>
     </gazebo>

File: urdf/robot.urdf.xacro (robot description, xacro)
@@ -2,4 +2,4 @@
 <robot xmlns:xacro="http://www.ros.org/wiki/xacro"  name="robot">
     <xacro:include filename="drivebase.xacro" />
-    <xacro:include filename="gazebo_control.xacro" />
+    <xacro:include filename="gz_ros2_control.xacro" />
 </robot>

Commit message: ros2_control simulation improvements

File: urdf/drivebase.xacro (robot description, xacro)
@@ -61,5 +61,5 @@
         <parent link="base_link"/>
         <child link="caster_wheel_FL"/>
-        <origin xyz="${caster_wheels_F_X_offset} ${caster_wheels_F_Y_spacing/2} ${-drive_wheel_radius + caster_wheel_radius + caster_wheel_Z_offset + 0.01}" rpy="0 0 0" />
+        <origin xyz="${caster_wheels_F_X_offset} ${caster_wheels_F_Y_spacing/2} ${-drive_wheel_radius + caster_wheel_radius + caster_wheel_Z_offset + 0.001}" rpy="0 0 0" />
     </joint>
     <xacro:caster_wheel name="caster_wheel_FR"></xacro:caster_wheel>
@@ -67,5 +67,5 @@
         <parent link="base_link"/>
         <child link="caster_wheel_FR"/>
-        <origin xyz="${caster_wheels_F_X_offset} -${caster_wheels_F_Y_spacing/2} ${-drive_wheel_radius + caster_wheel_radius + caster_wheel_Z_offset + 0.01}" rpy="0 0 0" />
+        <origin xyz="${caster_wheels_F_X_offset} -${caster_wheels_F_Y_spacing/2} ${-drive_wheel_radius + caster_wheel_radius + caster_wheel_Z_offset + 0.001}" rpy="0 0 0" />
     </joint>
     <xacro:caster_wheel name="caster_wheel_RL"></xacro:caster_wheel>
@@ -73,5 +73,5 @@
         <parent link="base_link"/>
         <child link="caster_wheel_RL"/>
-        <origin xyz="${caster_wheels_R_X_offset} ${caster_wheels_R_Y_spacing/2} ${-drive_wheel_radius + caster_wheel_radius + caster_wheel_Z_offset + 0.01}" rpy="0 0 0" />
+        <origin xyz="${caster_wheels_R_X_offset} ${caster_wheels_R_Y_spacing/2} ${-drive_wheel_radius + caster_wheel_radius + caster_wheel_Z_offset + 0.001}" rpy="0 0 0" />
     </joint>
     <xacro:caster_wheel name="caster_wheel_RR"></xacro:caster_wheel>
@@ -79,5 +79,5 @@
         <parent link="base_link"/>
         <child link="caster_wheel_RR"/>
-        <origin xyz="${caster_wheels_R_X_offset} -${caster_wheels_R_Y_spacing/2} ${-drive_wheel_radius + caster_wheel_radius + caster_wheel_Z_offset + 0.01}" rpy="0 0 0" />
+        <origin xyz="${caster_wheels_R_X_offset} -${caster_wheels_R_Y_spacing/2} ${-drive_wheel_radius + caster_wheel_radius + caster_wheel_Z_offset + 0.001}" rpy="0 0 0" />
     </joint>
 </robot>

File: urdf/params.xacro (robot description, xacro)
@@ -1,5 +1,5 @@
 <?xml version="1.0"?>
 <robot xmlns:xacro="http://www.ros.org/wiki/xacro">
-    <xacro:property name="drive_wheel_radius" value="0.17" /> <!-- TODO: Calibrate Drive wheel radius -->
+    <xacro:property name="drive_wheel_radius" value="0.1685" />
     <xacro:property name="drive_wheel_thickness" value="0.075" />
     <xacro:property name="caster_wheel_radius" value="0.075" />
@@ -12,5 +12,5 @@
     <xacro:property name="chassis_X_offset" value="-0.1" />
     <xacro:property name="chassis_Z_offset" value="0.08" />
-    <xacro:property name="drive_wheels_Y_spacing" value="0.46" />
+    <xacro:property name="drive_wheels_Y_spacing" value="0.54" />
     <xacro:property name="caster_wheels_F_Y_spacing" value="0.52" />
     <xacro:property name="caster_wheels_R_Y_spacing" value="0.405" />

File: urdf/robot.urdf.xacro (robot description, xacro)
@@ -1,7 +1,6 @@
 <?xml version="1.0"?>
 <robot xmlns:xacro="http://www.ros.org/wiki/xacro"  name="robot">
+    <xacro:arg name="sim_mode" default="false"/>
     <xacro:include filename="drivebase.xacro" />
-    <!-- TODO: Conditionally include either xacro -->
-    <!-- <xacro:include filename="gz_ros2_control.xacro" /> -->
     <xacro:include filename="ros2_control.xacro" />
 </robot>

File: urdf/ros2_control.xacro (robot description, xacro)
@@ -2,29 +2,81 @@
 <robot xmlns:xacro="http://www.ros.org/wiki/xacro">
     <xacro:include filename="params.xacro" />
-    <ros2_control name="DriveBaseSystem" type="system">
-        <hardware>
-            <plugin>luggage_av/LuggageAVHardawreInterface</plugin>
-            <param name="device">/dev/ttyS0</param>
-            <param name="linear_velocity_min">-3.233</param>
-            <param name="linear_velocity_max">3.233</param>
-            <param name="hardware_command_min">-8312</param>
-            <param name="hardware_command_max">8312</param>
-        </hardware>
-        <joint name="drive_wheel_L_joint">
-            <command_interface name="velocity">
-                <param name="min">-1.0</param>
-                <param name="max">1.0</param>
-            </command_interface>
-            <state_interface name="position"/>
-            <state_interface name="velocity"/>
-        </joint>
-        <joint name="drive_wheel_R_joint">
-            <command_interface name="velocity">
-                <param name="min">-1.0</param>
-                <param name="max">1.0</param>
-            </command_interface>
-            <state_interface name="position"/>
-            <state_interface name="velocity"/>
-        </joint>
-    </ros2_control>
+    <!-- TODO: Set params of each command interface such as min, max, initial value, etc -->
+    <xacro:unless value="$(arg sim_mode)">
+        <ros2_control name="DriveBaseSystem" type="system">
+            <hardware>
+                <plugin>luggage_av/LuggageAVHardawreInterface</plugin>
+                <param name="device">/dev/ttyS0</param>
+                <param name="linear_velocity_min">-3.233</param>
+                <param name="linear_velocity_max">3.233</param>
+                <param name="hardware_command_min">-8312</param>
+                <param name="hardware_command_max">8312</param>
+            </hardware>
+            <joint name="drive_wheel_L_joint">
+                <command_interface name="velocity">
+                    <param name="min">-1.0</param>
+                    <param name="max">1.0</param>
+                </command_interface>
+                <state_interface name="position"/>
+                <state_interface name="velocity"/>
+            </joint>
+            <joint name="drive_wheel_R_joint">
+                <command_interface name="velocity">
+                    <param name="min">-1.0</param>
+                    <param name="max">1.0</param>
+                </command_interface>
+                <state_interface name="position"/>
+                <state_interface name="velocity"/>
+            </joint>
+        </ros2_control>
+    </xacro:unless>
+    <xacro:if value="$(arg sim_mode)">
+        <ros2_control name="GazeboSimSystem" type="system">
+            <hardware>
+                <plugin>gz_ros2_control/GazeboSimSystem</plugin>
+            </hardware>
+            <joint name="drive_wheel_L_joint">
+                <command_interface name="velocity">
+                    <param name="min">-5</param>
+                    <param name="max">5</param>
+                </command_interface>
+                <state_interface name="position"/>
+                <state_interface name="velocity"/>
+            </joint>
+            <joint name="drive_wheel_R_joint">
+                <command_interface name="velocity">
+                    <param name="min">-5</param>
+                    <param name="max">5</param>
+                </command_interface>
+                <state_interface name="position"/>
+                <state_interface name="velocity"/>
+            </joint>
+        </ros2_control>
+        <gazebo>
+            <plugin filename="gz_ros2_control-system" name="gz_ros2_control::GazeboSimROS2ControlPlugin">
+                <parameters>$(find luggage_av)/parameters/controller_manager.yaml</parameters>
+                <parameters>$(find luggage_av)/parameters/gz_ros2_control.yaml</parameters>
+                <ros>
+                    <namespace>luggage_av</namespace>
+                    <remapping>/luggage_av/diff_drive_controller/cmd_vel:=/luggage_av/cmd_vel</remapping>
+                </ros>
+            </plugin>
+        </gazebo>
+        <gazebo reference="caster_wheel_FL">
+            <mu value="0.001" />
+            <mu2 value="0.001" />
+        </gazebo>
+        <gazebo reference="caster_wheel_FR">
+            <mu value="0.001" />
+            <mu2 value="0.001" />
+        </gazebo>
+        <gazebo reference="caster_wheel_RL">
+            <mu value="0.001" />
+            <mu2 value="0.001" />
+        </gazebo>
+        <gazebo reference="caster_wheel_RR">
+            <mu value="0.001" />
+            <mu2 value="0.001" />
+        </gazebo>
+    </xacro:if>
 </robot>

File: urdf/wheels.xacro (robot description, xacro)
@@ -12,5 +12,5 @@
         <link name="${name}">
             <visual>
-                <origin xyz="0 ${drive_wheel_thickness/2} 0" rpy="-${pi/2} 0 0" />
+                <origin xyz="0 0 0" rpy="-${pi/2} 0 0" />
                 <geometry>
                     <cylinder radius="${drive_wheel_radius}" length="${drive_wheel_thickness}" />
@@ -19,5 +19,5 @@
             </visual>
             <collision>
-                <origin xyz="0 ${drive_wheel_thickness/2} 0" rpy="-${pi/2} 0 0" />
+                <origin xyz="0 0 0" rpy="-${pi/2} 0 0" />
                 <geometry>
                     <cylinder radius="${drive_wheel_radius}" length="${drive_wheel_thickness}" />
@@ -25,5 +25,5 @@
             </collision>
             <xacro:inertial_cylinder mass="2.0" radius="${drive_wheel_radius}" length="${drive_wheel_thickness}">
-                <origin xyz="0 ${drive_wheel_thickness/2} 0" rpy="-${pi/2} 0 0" />
+                <origin xyz="0 0 0" rpy="-${pi/2} 0 0" />
             </xacro:inertial_cylinder>
         </link>
