Commit message: slam in gazebo

File: urdf/wheels.xacro (robot description, xacro)
@@ -21,5 +21,5 @@
                 <origin xyz="0 0 0" rpy="-${pi/2} 0 0" />
                 <geometry>
-                    <cylinder radius="${drive_wheel_radius}" length="${drive_wheel_thickness}" />
+                    <sphere radius="${drive_wheel_radius}" />
                 </geometry>
             </collision>
@@ -42,5 +42,5 @@
                 <origin xyz="-${caster_wheel_X_offset} 0 -${caster_wheel_Z_offset}" rpy="-${pi/2} 0 0" />
                 <geometry>
-                    <cylinder radius="${caster_wheel_radius}" length="${caster_wheel_thickness}"/>
+                    <sphere radius="${caster_wheel_radius}"/>
                 </geometry>
             </collision>
