Commit message: Added working lidar, but has drift

File: urdf/params.xacro (robot description, xacro)
@@ -17,3 +17,9 @@
     <xacro:property name="caster_wheels_F_X_offset" value="0.35" />
     <xacro:property name="caster_wheels_R_X_offset" value="-0.4" />
+    <!--LIDAR-->
+    <xacro:property name="lidar_pole_height" value="0.293" />
+    <xacro:property name="lidar_pole_width" value="0.0635" />
+    <xacro:property name="lidar_pole_length" value="0.0635" />
+    <xacro:property name="lidar_sensor_height" value="0.02794" />
+    <xacro:property name="lidar_sensor_radius" value="0.0635" />
 </robot>

File: urdf/robot.urdf.xacro (robot description, xacro)
@@ -4,3 +4,4 @@
     <xacro:include filename="drivebase.xacro" />
     <xacro:include filename="ros2_control.xacro" />
+    <xacro:include filename="lidar.xacro" />
 </robot>

Commit message: Camera URDF

File: urdf/params.xacro (robot description, xacro)
@@ -1,4 +1,5 @@
 <?xml version="1.0"?>
 <robot xmlns:xacro="http://www.ros.org/wiki/xacro">
+    <!-- WHEELS -->
     <xacro:property name="drive_wheel_radius" value="0.1685" />
     <xacro:property name="drive_wheel_thickness" value="0.075" />
@@ -7,4 +8,5 @@
     <xacro:property name="caster_wheel_X_offset" value="0.05" />
     <xacro:property name="caster_wheel_Z_offset" value="0.09" />
+    <!-- DRIVEBASE -->
     <xacro:property name="chassis_width" value="0.43" />
     <xacro:property name="chassis_length" value="0.55" />
@@ -29,3 +31,10 @@
     <xacro:property name="lidar_sensor_y_offset" value="-0.055" />
     <xacro:property name="lidar_sensor_z_offset" value="${0.003+lidar_pole_height}" />
+    <!-- CAMERA -->
+    <xacro:property name="camera_length" value="0.09" />
+    <xacro:property name="camera_width" value="0.024" />
+    <xacro:property name="camera_height" value="0.025" />
+    <xacro:property name="camera_x_offset" value="0" />
+    <xacro:property name="camera_y_offset" value="-0.071" />
+    <xacro:property name="camera_z_offset" value="${lidar_pole_height-0.06}" />
 </robot>

File: urdf/robot.urdf.xacro (robot description, xacro)
@@ -7,3 +7,4 @@
     <xacro:include filename="ros2_control.xacro" />
     <xacro:include filename="lidar.xacro" />
+    <xacro:include filename="camera.xacro" />
 </robot>
