Commit message: Camera GZ integration

File: urdf/camera.xacro (robot description, xacro)
@@ -8,22 +8,22 @@
         <parent link="lidar_mount_link"/>
         <child link="base_camera"/>
-        <origin xyz="${camera_x_offset} ${camera_y_offset} ${camera_z_offset}" rpy="0 0 ${pi/2}"/> <!--half the height of the mount + half the height of the lidar itself -->
+        <origin xyz="${camera_x_offset} ${camera_y_offset} ${camera_z_offset}" rpy="${-pi/2} 0 ${-pi/2}"/> <!--half the height of the mount + half the height of the lidar itself -->
     </joint>
     <link name="base_camera">
         <visual>
-            <origin xyz="0 ${camera_width/2} 0" rpy="0 0 0"/>
+            <origin xyz="0 0 ${-camera_width/2}" rpy="0 0 0"/>
             <geometry>
-                <box size="${camera_length} ${camera_width} ${camera_height}" />
+                <box size="${camera_length} ${camera_height} ${camera_width}" />
             </geometry>
             <material name="camera_black"/>
         </visual>
         <collision>
-            <origin xyz="0 ${camera_width/2} 0" rpy="0 0 0"/>
+            <origin xyz="0 0 ${-camera_width/2}" rpy="0 0 0"/>
             <geometry>
-                <box size="${camera_length} ${camera_width} ${camera_height}" />
+                <box size="${camera_length} ${camera_height} ${camera_width}" />
             </geometry>
         </collision>
-        <xacro:inertial_box mass="0.1" x="${camera_length}" y="${camera_width}" z="${camera_height}" >
-            <origin xyz="0 0 ${lidar_sensor_height/2}" rpy="0 0 0"/>
+        <xacro:inertial_box mass="0.1" x="${camera_length}" y="${camera_height}" z="${camera_width}" >
+            <origin xyz="0 0 ${-camera_width/2}" rpy="0 0 0"/>
         </xacro:inertial_box>
     </link>
@@ -31,8 +31,10 @@
         <material>Gazebo/Black</material>
         <sensor name="camera" type="camera">
-            <pose> 0 0 0 0 0 0 </pose>
+            <pose> 0 0 0 ${pi/2} ${-pi/2} 0</pose>
+            <always_on>true</always_on>
             <visualize>true</visualize>
             <update_rate>30</update_rate>
-            <camera>
+            <camera name="logitech_c920">
+                <camera_info_topic>camera_info</camera_info_topic>
                 <horizontal_fov>1.229061</horizontal_fov>
                 <image>
@@ -46,7 +48,6 @@
                 </clip>
             </camera>
-            <plugin name="camera_controller" filename="libgazebo_ros_camera.so">
-                <frame_name>camera_link_optical</frame_name>
-            </plugin>
+            <topic>/$(arg namespace)/image_raw</topic>
+            <gz_frame_id>$(arg namespace)/base_camera</gz_frame_id>
         </sensor>
     </gazebo>
