Commit message: Fixed worlds args and lidar location

File: urdf/lidar.xacro (robot description, xacro)
@@ -8,11 +8,11 @@
         <color rgba="0.2 0.2 1 1"/>
     </material>
-    <xacro:property name="lidar_pole_x_origin" value="${chassis_length/2}" />
-    <xacro:property name="lidar_pole_y_origin" value="${-chassis_width/2}" />
+    <xacro:property name="lidar_pole_x_origin" value="${-chassis_length/2}" />
+    <xacro:property name="lidar_pole_y_origin" value="${chassis_width/2}" />
     <xacro:property name="lidar_pole_z_origin" value="${chassis_height - drive_wheel_radius + chassis_Z_offset}" />
     <joint name="lidar_mount_joint" type="fixed">
         <parent link="base_link"/>
         <child link="lidar_mount_link"/>
-        <origin xyz = "${lidar_pole_x_origin-lidar_pole_length/2 + chassis_X_offset} ${lidar_pole_y_origin+lidar_pole_width/2} ${lidar_pole_z_origin + lidar_pole_height/2}"/>
+        <origin xyz = "${lidar_pole_x_origin+lidar_pole_length/2 + chassis_X_offset} ${lidar_pole_y_origin-lidar_pole_width/2} ${lidar_pole_z_origin + lidar_pole_height/2}"/>
     </joint>
     <link name="lidar_mount_link">

Commit message: local costmap, additional rviz improvements, namespaced_tf in some launch files

File: urdf/lidar.xacro (robot description, xacro)
@@ -37,8 +37,8 @@
     <joint name="laser_joint" type="fixed">
         <parent link="lidar_mount_link"/>
-        <child link="laser"/>
+        <child link="base_laser"/>
         <origin xyz = "0 0 ${(lidar_pole_height+lidar_sensor_height)/2}"/> <!--half the height of the mount + half the height of the lidar itself -->
     </joint>
-    <link name="laser">
+    <link name="base_laser">
         <visual>
             <geometry>
@@ -56,7 +56,7 @@
         </xacro:inertial_cylinder>
     </link>
-    <gazebo reference="laser">
+    <gazebo reference="base_laser">
         <material>Gazebo/blue</material>
-        <sensor name="laser" type="gpu_lidar">
+        <sensor name="lidar" type="gpu_lidar">
             <pose> 0 0 0 0 0 0 </pose>
             <visualize>false</visualize>
@@ -76,5 +76,5 @@
             </lidar>
             <topic>/luggage_av/scan</topic>
-            <gz_frame_id>luggage_av/laser</gz_frame_id>
+            <gz_frame_id>luggage_av/base_laser</gz_frame_id>
         </sensor>
     </gazebo>

Commit message: Fix lidar positioning

File: urdf/lidar.xacro (robot description, xacro)
@@ -5,18 +5,15 @@
         <color rgba="0 0 0 1"/>
     </material>
-    <material name="lidar_blue">
-        <color rgba="0.2 0.2 1 1"/>
+    <material name="lidar_burgundy">
+        <color rgba="0.5 0 0.125 0.8"/>
     </material>
-    <xacro:property name="lidar_pole_x_origin" value="${-chassis_length/2}" />
-    <xacro:property name="lidar_pole_y_origin" value="${chassis_width/2}" />
-    <xacro:property name="lidar_pole_z_origin" value="${chassis_height - drive_wheel_radius + chassis_Z_offset}" />
     <joint name="lidar_mount_joint" type="fixed">
         <parent link="base_link"/>
         <child link="lidar_mount_link"/>
-        <origin xyz = "${lidar_pole_x_origin+lidar_pole_length/2 + chassis_X_offset} ${lidar_pole_y_origin-lidar_pole_width/2} ${lidar_pole_z_origin + lidar_pole_height/2}"/>
+        <origin xyz = "${lidar_pole_x_offset} ${lidar_pole_y_offset} ${lidar_pole_z_offset}"/>
     </joint>
     <link name="lidar_mount_link">
         <visual>
-            <origin xyz = "0 0 0"/>
+            <origin xyz="${-lidar_pole_length/2} ${-lidar_pole_width/2} ${lidar_pole_height/2}" rpy="0 0 0"/>
             <geometry>
                 <box size="${lidar_pole_length} ${lidar_pole_width} ${lidar_pole_height}"/>
@@ -25,5 +22,5 @@
         </visual>
         <collision>
-            <origin xyz = "0 0 0"/>
+            <origin xyz="${-lidar_pole_length/2} ${-lidar_pole_width/2} ${lidar_pole_height/2}" rpy="0 0 0"/>
             <geometry>
                 <box size="${lidar_pole_length} ${lidar_pole_width} ${lidar_pole_height}"/>
@@ -32,5 +29,5 @@
         </collision>
         <xacro:inertial_box mass="0.1" x="${lidar_pole_length}" y="${lidar_pole_width}" z="${lidar_pole_height}">
-            <origin xyz="0 0 0" rpy="0 0 0"/>
+            <origin xyz="${-lidar_pole_length/2} ${-lidar_pole_width/2} ${lidar_pole_height/2}" rpy="0 0 0"/>
         </xacro:inertial_box>
     </link>
@@ -38,14 +35,16 @@
         <parent link="lidar_mount_link"/>
         <child link="base_laser"/>
-        <origin xyz = "0 0 ${(lidar_pole_height+lidar_sensor_height)/2}"/> <!--half the height of the mount + half the height of the lidar itself -->
+        <origin xyz="${lidar_sensor_x_offset} ${lidar_sensor_y_offset} ${lidar_sensor_z_offset}" rpy="0 0 ${pi/2}"/> <!--half the height of the mount + half the height of the lidar itself -->
     </joint>
     <link name="base_laser">
         <visual>
+            <origin xyz="0 0 ${lidar_sensor_height/2}" rpy="0 0 0"/>
             <geometry>
                 <cylinder radius="${lidar_sensor_radius}" length="${lidar_sensor_radius}"/>
             </geometry>
-            <material name="lidar_blue"/>
+            <material name="lidar_burgundy"/>
         </visual>
         <collision>
+            <origin xyz="0 0 ${lidar_sensor_height/2}" rpy="0 0 0"/>
             <geometry>
                 <cylinder radius="${lidar_sensor_radius}" length="${lidar_sensor_radius}"/>
@@ -53,5 +52,5 @@
         </collision>
         <xacro:inertial_cylinder mass="0.1" radius="${lidar_sensor_radius}" length="${lidar_sensor_radius}" >
-            <origin xyz="0 0 ${(lidar_pole_height+lidar_sensor_height)/2}" rpy="0 0 0"/>
+            <origin xyz="0 0 ${lidar_sensor_height/2}" rpy="0 0 0"/>
         </xacro:inertial_cylinder>
     </link>

File: urdf/params.xacro (robot description, xacro)
@@ -18,8 +18,14 @@
     <xacro:property name="caster_wheels_R_X_offset" value="-0.4" />
     <!--LIDAR-->
-    <xacro:property name="lidar_pole_height" value="0.293" />
-    <xacro:property name="lidar_pole_width" value="0.0635" />
-    <xacro:property name="lidar_pole_length" value="0.0635" />
-    <xacro:property name="lidar_sensor_height" value="0.02794" />
-    <xacro:property name="lidar_sensor_radius" value="0.0635" />
+    <xacro:property name="lidar_pole_length" value="0.04" />
+    <xacro:property name="lidar_pole_width" value="0.02" />
+    <xacro:property name="lidar_pole_height" value="0.449" />
+    <xacro:property name="lidar_pole_x_offset" value="-0.2794" />
+    <xacro:property name="lidar_pole_y_offset" value="${0.1397+0.102}" />
+    <xacro:property name="lidar_pole_z_offset" value="${0.365-drive_wheel_radius}" />
+    <xacro:property name="lidar_sensor_height" value="0.04" />
+    <xacro:property name="lidar_sensor_radius" value="0.0375" />
+    <xacro:property name="lidar_sensor_x_offset" value="-0.01" />
+    <xacro:property name="lidar_sensor_y_offset" value="-0.055" />
+    <xacro:property name="lidar_sensor_z_offset" value="${0.003+lidar_pole_height}" />
 </robot>

Commit message: Revert "Ee drive in local square demo"

File: urdf/lidar.xacro (robot description, xacro)
@@ -37,8 +37,8 @@
     <joint name="laser_joint" type="fixed">
         <parent link="lidar_mount_link"/>
-        <child link="base_laser"/>
+        <child link="laser"/>
         <origin xyz = "0 0 ${(lidar_pole_height+lidar_sensor_height)/2}"/> <!--half the height of the mount + half the height of the lidar itself -->
     </joint>
-    <link name="base_laser">
+    <link name="laser">
         <visual>
             <geometry>
@@ -56,7 +56,7 @@
         </xacro:inertial_cylinder>
     </link>
-    <gazebo reference="base_laser">
+    <gazebo reference="laser">
         <material>Gazebo/blue</material>
-        <sensor name="lidar" type="gpu_lidar">
+        <sensor name="laser" type="gpu_lidar">
             <pose> 0 0 0 0 0 0 </pose>
             <visualize>false</visualize>
@@ -75,6 +75,6 @@
                 </range>
             </lidar>
-            <topic>scan</topic>
-            <gz_frame_id>$(arg namespace)/base_laser</gz_frame_id>
+            <topic>/luggage_av/scan</topic>
+            <gz_frame_id>luggage_av/laser</gz_frame_id>
         </sensor>
     </gazebo>

File: urdf/robot.urdf.xacro (robot description, xacro)
@@ -2,5 +2,4 @@
 <robot xmlns:xacro="http://www.ros.org/wiki/xacro"  name="robot">
     <xacro:arg name="sim_mode" default="false"/>
-    <xacro:arg name="namespace" default="luggage_av"/>
     <xacro:include filename="drivebase.xacro" />
     <xacro:include filename="ros2_control.xacro" />

File: urdf/ros2_control.xacro (robot description, xacro)
@@ -56,6 +56,8 @@
             <plugin filename="gz_ros2_control-system" name="gz_ros2_control::GazeboSimROS2ControlPlugin">
                 <parameters>$(find luggage_av)/parameters/controller_manager.yaml</parameters>
+                <parameters>$(find luggage_av)/parameters/gz_ros2_control.yaml</parameters>
                 <ros>
-                    <namespace>/$(arg namespace)</namespace>
+                    <namespace>luggage_av</namespace>
+                    <remapping>/luggage_av/diff_drive_controller/cmd_vel:=/luggage_av/cmd_vel</remapping>
                 </ros>
             </plugin>

Commit message: FIx lidar dimensions and offsets

File: urdf/lidar.xacro (robot description, xacro)
@@ -35,5 +35,5 @@
         <parent link="lidar_mount_link"/>
         <child link="base_laser"/>
-        <origin xyz="${lidar_sensor_x_offset} ${lidar_sensor_y_offset} ${lidar_sensor_z_offset}" rpy="0 0 ${pi/2}"/> <!--half the height of the mount + half the height of the lidar itself -->
+        <origin xyz="${lidar_sensor_x_offset} ${lidar_sensor_y_offset} ${lidar_sensor_z_offset}" rpy="0 0 ${pi}"/> <!--half the height of the mount + half the height of the lidar itself -->
     </joint>
     <link name="base_laser">

File: urdf/params.xacro (robot description, xacro)
@@ -18,14 +18,14 @@
     <xacro:property name="caster_wheels_R_X_offset" value="-0.4" />
     <!--LIDAR-->
-    <xacro:property name="lidar_pole_length" value="0.04" />
-    <xacro:property name="lidar_pole_width" value="0.02" />
-    <xacro:property name="lidar_pole_height" value="0.449" />
-    <xacro:property name="lidar_pole_x_offset" value="-0.2794" />
-    <xacro:property name="lidar_pole_y_offset" value="${0.1397+0.102}" />
+    <xacro:property name="lidar_pole_length" value="0.0365" />
+    <xacro:property name="lidar_pole_width" value="0.0365" />
+    <xacro:property name="lidar_pole_height" value="1.041" />
+    <xacro:property name="lidar_pole_x_offset" value="-0.267" />
+    <xacro:property name="lidar_pole_y_offset" value="0.254" />
     <xacro:property name="lidar_pole_z_offset" value="${0.365-drive_wheel_radius}" />
     <xacro:property name="lidar_sensor_height" value="0.04" />
     <xacro:property name="lidar_sensor_radius" value="0.0375" />
-    <xacro:property name="lidar_sensor_x_offset" value="-0.01" />
-    <xacro:property name="lidar_sensor_y_offset" value="-0.055" />
-    <xacro:property name="lidar_sensor_z_offset" value="${0.003+lidar_pole_height}" />
+    <xacro:property name="lidar_sensor_x_offset" value="0.0254" />
+    <xacro:property name="lidar_sensor_y_offset" value="${-lidar_pole_width/2}" />
+    <xacro:property name="lidar_sensor_z_offset" value="1.067" />
 </robot>
